File: Aurora Orbiton Edition/Aurora Orbiton Edition.kicad_sch (KiCad schematic)
At the start: 154 parts, among them IC1 TPS259830LNRGER, J1 Radio4Pin, J10 Pyro8Pin, J11 Power8Pin, J2 USB_C_Receptacle_USB2.0_14P, J3 GPS7Pin, J4 GPIO4Pin, J6 QWIIC I2C, J8 SPI9Pin, J9 Prog5Pin, M1 Motor_Servo, M2 Motor_Servo, M3 Motor_Servo, M4 Motor_Servo, M5 Motor_Servo, M6 Motor_Servo, M7 Motor_Servo, M8 Motor_Servo, Q1 Si7617DN, SW1 SW_SPDT, SW2 SW_Push, U1 TVS0500DRV, U10 UCS3205, U11 UCS3205, U12 UCS3205, U2 AP63203WU, U3 STM32H753VITx, U4 BMP390L, U5 BMI088, U6 H3LIS331DLTR, U7 W25Q128JVS, U8 DRV8871DDA, U9 UCS3205, Y1 C13740

Commit message: Updated to R2, unchecked
Parts:
- added SW1: SW_Push, Button_Switch_SMD:SW_Push_SPST_NO_Alps_SKRK, symbol Switch:SW_Push
- renumbered C20 to C19, C21 to C20, C24 to C21, C25 to C22, C22 to C23, C23 to C24, C26 to C25, C27 to C26, C28 to C27, C29 to C28, C30 to C29, C31 to C30, C32 to C31, C33 to C32, C34 to C33, C35 to C34, C36 to C35, C37 to C36, C38 to C37, C39 to C38, C40 to C39, C41 to C40, C42 to C41, C43 to C42, C44 to C43, C45 to C44, C46 to C45, C47 to C46, C48 to C47, C49 to C48, J6 to J5, J8 to J6, J11 to J7, J9 to J8, J10 to J9, R16 to R15, R15 to R16, R19 to R18, R20 to R19, R21 to R20, R22 to R21, R23 to R22, R24 to R23, R25 to R24, R26 to R25, R27 to R26, R28 to R27, R29 to R28, R30 to R29, R31 to R30, R32 to R31, R33 to R32, R34 to R33, R35 to R34, R36 to R35, R37 to R36, R38 to R37, R39 to R38, R40 to R39, R41 to R40, R42 to R41, R43 to R42, R44 to R43, R45 to R44, R46 to R45, R47 to R46, R48 to R47, R49 to R48, R50 to R49, R51 to R50, R52 to R51, R53 to R52, R54 to R53, R55 to R54, R56 to R55, SW1 to SW2, SW2 to SW3, U6 to U5, U5 to U6
Connections:
- net +3.3V: now also SW1.2
- net BOOT0: now also SW1.1
Other:
- moved on the sheet: R1
